File: BulkDispense/MAXIExpansionBoard/MAXIExpansionBoard.kicad_pcb (KiCad board)
At the start: 2 copper layers, 57.2 x 100 mm, 25 parts, among them J1 BS1~4, J10 FS3, J11 R6~R7, J12 R8~R9, J13 OS1~4, J14 WV1~2, J15 FS2, J16 FS4, J17 Analog Inputs, J18 Digital IN + R0~R4, J19 Digital Outputs, J2 MV1~4, J20 R4~R9, J21 Flow Sensors, J3 WB/WL, J4 PS/PCV, J5 Screw_Terminal_01x02, J6 R0~R1, J7 R2~R3, J8 R4~R5, J9 FS1

Commit message: Add STEP files
Parts:
- added kibuzzard-684C282C: G***, kibuzzard-684C282C, F.Cu at (125.0, 63.4)
- added kibuzzard-684C2929: G***, kibuzzard-684C2929, F.Cu at (125.0, 78.2)
- added kibuzzard-684C293C: G***, kibuzzard-684C293C, F.Cu at (125.0, 93.4)
- added kibuzzard-684C2942: G***, kibuzzard-684C2942, F.Cu at (125.0, 108.6)
- added kibuzzard-684C2947: G***, kibuzzard-684C2947, F.Cu at (125.0, 124.0)
- moved J3 3.77 mm to (143.0, 132.4), turned to 0 degrees
Routing:
- net /AI4: track 40.4 -> 32.1 mm
- net /AI7: track 28.7 -> 34.7 mm, vias 0 -> 1
- net /AI5: track 34.5 -> 32.6 mm
- net /FS1-1: track 55.1 -> 56.5 mm
- net /AI0: track 68.3 -> 69.5 mm
- net /AI1: track 58.8 -> 59.6 mm
- net /R2_OUT: track 26.9 -> 27.7 mm
- net /FS2-2: track 31.4 -> 32.3 mm
- net /R3_OUT: track 29.3 -> 30.1 mm
- net /FS3-1: track 40.8 -> 41.6 mm
- net /FS2-3: track 35.1 -> 35.9 mm
- net /DO3: track 46.1 -> 46.9 mm
- net /R8_OUT: track 22.2 -> 23.0 mm
- net /R7_OUT: track 11.2 -> 11.9 mm
- net /R5_IN: track 51.2 -> 51.9 mm
