File: LynxActuator/75v.kicad_sch (KiCad schematic)
At the start: 4 parts, among them M2 Motor_DC

Commit message: Visual Edits
Other:
- note added: "75V System"
Changed lines of the file:
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@@
+		)
+	)
+	(text "75V System"
+		(exclude_from_sim no)
+		(at 49.276 22.86 0)
+		(effects
+			(font
+				(size 5.08 5.08)
+			)
 		)
 	)
