File: LynxActuator/LynxActuator_expanded.kicad_sch (KiCad schematic)
At the start: 29 parts, among them J1 MIL-20 Connector, M1 Motor_DC, SW1 E-STOP, U1 ELR1-SC-24DC

Commit message: Visual Edits
Parts:
- removed CC3, CC5: CLEAR-CORE, symbol LynxActuatorSymbols:CLEAR-CORE
- removed CC4, CC6: CCIO-8, symbol LynxActuatorSymbols:CCIO-8
- removed EN2, EN3: CL-ENCDR-DFIN, symbol LynxActuatorSymbols:CL-ENCDR-DFIN
Connections:
- new net: TB1. (COM), TB3. (COM) (x3)
- new net: TB2. (COM), TB4. (COM) (x3)
- no-connect marks 27 -> 21
Other:
- removed sheet SENSORS
- note removed: "ClearCore Expansion Board"
- note removed: "Knob Encoder"
- note removed: "Sensor 1~4 Terminal Block"
- moved on the sheet: TB6
