File: LynxActuator/ac_supply.kicad_sch (KiCad schematic)
At the start: 3 parts

Commit message: Visual Edits
Other:
- note added: "AC Supply"
Changed lines of the file:
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@@
 	(generator_version "9.0")
 	(paper "User" 152.4 152.4)
+	(rectangle
+		(start 21.59 26.67)
+		(end 134.62 100.33)
+		(stroke
+			(width 0)
+			(type dash)
+		)
+		(fill
+			(type none)
+		)
+	)
+	(text "AC Supply"
+		(exclude_from_sim no)
+		(at 40.64 20.574 0)
+		(effects
+			(font
+				(size 5.08 5.08)
+			)
+		)
+	)
 	(junction
 		(at 83.82 67.31)
