File: LynxActuator/controllers.kicad_sch (KiCad schematic)
At the start: 3 parts

Commit message: Visual Edits
Connections:
- net MYSTERY_MOTOR renamed RAIL_MOTOR
- net MYSTERY_SENSOR renamed PRESSURE_SENSOR
Other:
- note added: "Controllers"
Changed lines of the file:
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@@
 		)
 	)
+	(text "Controllers"
+		(exclude_from_sim no)
+		(at 38.1 18.542 0)
+		(effects
+			(font
+				(size 5.08 5.08)
+			)
+		)
+	)
 	(text "ClearCore \nExpansion Board"
 		(exclude_from_sim no)
@@
 		)
 	)
-	(hierarchical_label "MYSTERY_SENSOR"
-		(shape input)
-		(at 195.58 93.98 0)
-		(effects
-			(font
-				(size 1.27 1.27)
-				(thickness 0.254)
-				(bold yes)
-				(color 107 0 255 1)
-			)
-			(justify left)
-		)
-	)
 	(hierarchical_label "SENSOR8_OUT"
 		(shape input)
@@
 		)
 	)
-	(hierarchical_label "GND_(CLEAR-CORE)"
+	(hierarchical_label "PRESSURE_SENSOR"
 		(shape input)
-		(at 162.56 130.81 180)
+		(at 195.58 93.98 0)
 		(effects
 			(font
 				(size 1.27 1.27)
 			)
-			(justify right)
+			(justify left)
 		)
 	)
-	(hierarchical_label "SENSOR7_OUT"
+	(hierarchical_label "GND_(CLEAR-CORE)"
 		(shape input)
-		(at 162.56 101.6 180)
+		(at 162.56 130.81 180)
 		(effects
 			(font
@@
 		)
 	)
-	(hierarchical_label "SENSOR10_OUT"
+	(hierarchical_label "SENSOR7_OUT"
 		(shape input)
-		(at 93.98 109.22 180)
+		(at 162.56 101.6 180)
 		(effects
 			(font
@@
 		)
 	)
-	(hierarchical_label "MYSTERY_MOTOR"
+	(hierarchical_label "SENSOR10_OUT"
 		(shape input)
-		(at 199.39 116.84 0)
+		(at 93.98 109.22 180)
 		(effects
 			(font
 				(size 1.27 1.27)
-				(thickness 0.254)
-				(bold yes)
-				(color 107 0 255 1)
 			)
-			(justify left)
+			(justify right)
 		)
 	)
@@
 		)
 	)
+	(hierarchical_label "RAIL_MOTOR"
+		(shape input)
+		(at 199.39 116.84 0)
+		(effects
+			(font
+				(size 1.27 1.27)
+			)
+			(justify left)
+		)
+	)
