File: LynxActuator/24v.kicad_sch (KiCad schematic)
At the start: 2 parts

Commit message: Visual Edits
Other:
- note added: "24V Power Distribuition"
Changed lines of the file:
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@@
+		)
+	)
+	(text "24V Power Distribuition"
+		(exclude_from_sim no)
+		(at 60.452 23.368 0)
+		(effects
+			(font
+				(size 5.08 5.08)
+			)
 		)
 	)

Commit message: Add updated layout
Connections:
- net +24V_(ST) is gone; now on net +24V_(LYNX_OUTBOUND): TB2.5
- net -24V_(ST) is gone; now on net -24V_(LYNX_OUTBOUND): TB1.6
- net +24V_(E-STOP): now also TB2.6; no longer TB2.7
- net +24V_(LYNX_OUTBOUND): no longer TB2.6
- net -24V_(LYNX_OUTBOUND): no longer TB1.7
Changed lines of the file:
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@@
+		)
+	)
+	(hierarchical_label "+24V_(CC)"
+		(shape input)
+		(at 43.18 81.28 180)
+		(effects
+			(font
+				(size 1.27 1.27)
+			)
+			(justify right)
+		)
+	)
+	(hierarchical_label "-24V_(LYNX_OUTBOUND)"
+		(shape input)
+		(at 116.84 91.44 180)
+		(effects
+			(font
+				(size 1.27 1.27)
+			)
+			(justify right)
+		)
+	)
+	(hierarchical_label "-24V"
+		(shape input)
+		(at 132.08 69.85 180)
+		(effects
+			(font
+				(size 1.27 1.27)
+			)
+			(justify right)
+		)
+	)
+	(hierarchical_label "-24V_(CC)"
+		(shape input)
+		(at 116.84 83.82 180)
+		(effects
+			(font
+				(size 1.27 1.27)
+			)
+			(justify right)
+		)
+	)
+	(hierarchical_label "+24V_(CCIO)"
+		(shape input)
+		(at 43.18 85.09 180)
+		(effects
+			(font
+				(size 1.27 1.27)
+			)
+			(justify right)
+		)
+	)
+	(hierarchical_label "-24V_(PH)"
+		(shape input)
+		(at 116.84 80.01 180)
+		(effects
+			(font
+				(size 1.27 1.27)
+			)
+			(justify right)
+		)
+	)
+	(hierarchical_label "-24V_(CT)"
+		(shape input)
+		(at 116.84 76.2 180)
+		(effects
+			(font
+				(size 1.27 1.27)
+			)
+			(justify right)
+		)
+	)
+	(hierarchical_label "+24V_(E-STOP)"
+		(shape input)
+		(at 43.18 92.71 180)
+		(effects
+			(font
+				(size 1.27 1.27)
+			)
+			(justify right)
 		)
 	)
 	(hierarchical_label "+24V_(LYNX_OUTBOUND)"
 		(shape input)
-		(at 43.18 92.71 180)
-		(effects
-			(font
-				(size 1.27 1.27)
-			)
-			(justify right)
-		)
-	)
-	(hierarchical_label "+24V_(CC)"
-		(shape input)
-		(at 43.18 81.28 180)
-		(effects
-			(font
-				(size 1.27 1.27)
-			)
-			(justify right)
-		)
-	)
-	(hierarchical_label "+24V_(ST)"
-		(shape input)
 		(at 43.18 88.9 180)
 		(effects
@@
 		)
 	)
-	(hierarchical_label "-24V"
-		(shape input)
-		(at 132.08 69.85 180)
-		(effects
-			(font
-				(size 1.27 1.27)
-			)
-			(justify right)
-		)
-	)
-	(hierarchical_label "-24V_(LYNX_OUTBOUND)"
-		(shape input)
-		(at 116.84 95.25 180)
-		(effects
-			(font
-				(size 1.27 1.27)
-			)
-			(justify right)
-		)
-	)
-	(hierarchical_label "-24V_(CC)"
-		(shape input)
-		(at 116.84 83.82 180)
-		(effects
-			(font
-				(size 1.27 1.27)
-			)
-			(justify right)
-		)
-	)
-	(hierarchical_label "+24V_(CCIO)"
-		(shape input)
-		(at 43.18 85.09 180)
-		(effects
-			(font
-				(size 1.27 1.27)
-			)
-			(justify right)
-		)
-	)
-	(hierarchical_label "-24V_(PH)"
-		(shape input)
-		(at 116.84 80.01 180)
-		(effects
-			(font
-				(size 1.27 1.27)
-			)
-			(justify right)
-		)
-	)
-	(hierarchical_label "+24V_(E-STOP)"
-		(shape input)
-		(at 43.18 96.52 180)
-		(effects
-			(font
-				(size 1.27 1.27)
-			)
-			(justify right)
-		)
-	)
-	(hierarchical_label "-24V_(CT)"
-		(shape input)
-		(at 116.84 76.2 180)
-		(effects
-			(font
-				(size 1.27 1.27)
-			)
-			(justify right)
-		)
-	)
 	(hierarchical_label "+24V_(PH)"
 		(shape input)
 		(at 43.18 77.47 180)
-		(effects
-			(font
-				(size 1.27 1.27)
-			)
-			(justify right)
-		)
-	)
-	(hierarchical_label "-24V_(ST)"
-		(shape input)
-		(at 116.84 91.44 180)
 		(effects
 			(font
@@
 			)
 		)
-		(property "Datasheet" ""
+		(property "Datasheet" "https://www.digikey.com/en/products/detail/phoenix-contact/3273110/7596951"
 			(at 132.08 88.9 0)
 			(effects
@@
 			)
 		)
-		(property "Datasheet" ""
+		(property "Datasheet" "https://www.digikey.com/en/products/detail/phoenix-contact/3273110/7596951"
 			(at 58.42 92.71 0)
 			(effects
