File: LynxActuator/25v_power_supply.kicad_sch (KiCad schematic)
At the start: 2 parts

Commit message: Visual Edits
Other:
- note added: "24V Power Supply"
Changed lines of the file:
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@@
+		)
+	)
+	(text "24V Power Supply"
+		(exclude_from_sim no)
+		(at 50.8 23.368 0)
+		(effects
+			(font
+				(size 5.08 5.08)
+			)
 		)
 	)

Commit message: Add updated layout
Parts:
- TB4: value PTTB_2,5 -> 277-17721-ND
Other:
- note removed: "Mystery Part"
Changed lines of the file:
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@@
 		)
 	)
-	(text "Mystery Part"
-		(exclude_from_sim no)
-		(at 82.804 65.2385 0)
-		(effects
-			(font
-				(size 1.27 1.27)
-				(thickness 0.254)
-				(bold yes)
-				(color 107 0 255 1)
-			)
-		)
-	)
 	(junction
 		(at 92.71 78.7005)
@@
 		(dnp no)
 		(property "Reference" "TB4"
-			(at 82.296 67.5245 0)
+			(at 82.55 64.008 0)
 			(effects
 				(font
@@
 			)
 		)
-		(property "Value" "PTTB_2,5"
+		(property "Value" "277-17721-ND"
 			(at 82.296 66.5085 0)
 			(effects
@@
 					(size 1.27 1.27)
 				)
-				(hide yes)
 			)
 		)
@@
 			)
 		)
-		(property "Datasheet" "https://www.phoenixcontact.com/en-us/products/multi-level-terminal-block-pttb-25-3210567"
+		(property "Datasheet" "https://www.digikey.com/en/products/detail/phoenix-contact/2908262/9448966?gad_source=1&gad_campaignid=20228387720&gbraid=0AAAAADrbLlho9EFuX5hIKj-tWfql-IRh7&gclid=Cj0KCQjwjdTCBhCLARIsAEu8bpJGTFnnMFEty_f8fJ23Np9g4PNZFmSv_RjYYWPvjP4daSlmclphF3EaAkU8EALw_wcB&gclsrc=aw.ds"
 			(at 82.55 72.3505 0)
 			(effects
