File: LynxActuator/sensors.kicad_sch (KiCad schematic)
At the start: 5 parts, among them J2 MIL-20 Connector

Commit message: Visual Edits
Connections:
- new net: TB13. (COM), TB14. (COM) (x3)
- new net: TB15. (COM), TB16. (COM) (x3)
Other:
- note added: "Sensors"
- moved on the sheet: J2, TB13, TB14, TB15, TB16

Commit message: Add updated layout
Parts:
- removed TB13, TB14, TB15, TB16: WAGO 2000-5420/1399-987, symbol LynxActuatorSymbols:WAGO-2000-5420
Connections:
- no-connect marks 17 -> 0
Other:
- note removed: "Sensor 1~4 Terminal Block"
- moved on the sheet: J2
