File: BulkDispense/BreakoutBoard/BreakoutBoard.kicad_pcb (KiCad board)
At the start: 2 copper layers, 80 x 80 mm, 74 parts, among them J1 PS, J11 WL1, J12 WL2, J15 WB1, J16 WB2, J20 LDS, J24 WB-MV1, J36 WB-MV2, J37 RV1, J38 RV3, J39 RV2, J4 Signal, J40 RV4, J41 MV1, J42 MV2, J43 MV3, J44 MV4, J45 WB-MV1, J46 WB-MV3, J47 WB-MV2, J48 WB-MV4, J5 PCV, U1 TCA9548APWR, U2 LMR51430, U3 LMR51430, U4 TVS2700DRV

Commit message: Final Update
Parts:
- C1: footprint Capacitor_SMD:C_01005_0402Metric -> Capacitor_SMD:C_0402_1005Metric
- D1, D3, D4: footprint LED_SMD:LED_0201_0603Metric -> LED_SMD:LED_0603_1608Metric
- R1: footprint Resistor_SMD:R_0805_2012Metric -> Resistor_SMD:R_1206_3216Metric
- R3, R4: footprint Resistor_SMD:R_0805_2012Metric -> Resistor_SMD:R_0603_1608Metric
- moved R1 1.73 mm to (128.6, 50.4)
- moved D3 0.40 mm to (173.6, 31.4)
- moved C1 0.15 mm to (116.5, 45.4)
- moved D4 0.15 mm to (154.5, 31.8)
- renumbered FS4 to J10, FS3 to J13, FS2 to J14, FS1 to J17
Routing:
- net GND: track 29.5 -> 31.5 mm
- net Net-(D1-K): track 1.85 -> 2.37 mm
